Commit message: control et odom

File: install/roboto/share/roboto/robo_description/urdf/chassi/robot.urdf.xacro (robot description, xacro)
@@ -13,10 +13,10 @@
         <mesh filename="package://roboto/robo_description/urdf/chassi/support.stl"/>
         </geometry>
-        <material name="support_material">
-        <color rgba="0.2313725490196078538 0.38039215686274507888 0.38 1.0"/>
+        <material name="body-material">
+        <color rgba="1 1 1 1 "/>
         </material>
     </visual>
     <collision>
-        <origin xyz="0.12499999999999995837 -0.12500000000000002776 1.3877787807814456755e-17" rpy="0 -0 0" />
+        <origin xyz="0.12499999999999995837 -0.12500000000000002776 1.3877787807814456755e-17" rpy="0 0 0" />
         <geometry>
         <mesh filename="package://roboto/robo_description/urdf/chassi/support.stl"/>
@@ -24,14 +24,14 @@
     </collision>
     <visual>
-        <origin xyz="0.12499999999999998612 -0.12500000000000002776 0" rpy="0 -0 0" />
+        <origin xyz="0.12499999999999998612 -0.12500000000000002776 0" rpy="0 0 0" />
         <geometry>
         <mesh filename="package://roboto/robo_description/urdf/chassi/body.stl"/>
         </geometry>
         <material name="body_material">
-        <color rgba="0.61568627450980395466 0.81176470588235294379 0.92941176470588238168 1.0"/>
+        <color rgba="1 1 1 1 "/>
         </material>
     </visual>
     <collision>
-        <origin xyz="0.12499999999999998612 -0.12500000000000002776 0" rpy="0 -0 0" />
+        <origin xyz="0.12499999999999998612 -0.12500000000000002776 0" rpy="0 0 0" />
         <geometry>
         <mesh filename="package://roboto/robo_description/urdf/chassi/body.stl"/>
@@ -68,5 +68,5 @@
     </link>
     <joint name="${name}_joint" type="continuous">
-      <parent link="base_link"/>
+      <parent link="body"/>
       <child link="${name}_link"/>
       <origin xyz="${x} ${y} ${z}" rpy="${rpy}"/>
@@ -78,31 +78,5 @@
   <xacro:wheel name="wheel_3" x="-0.12" y="-0.12" z="0.015" rpy="${pi/2}  0  ${3*pi/4}"/>
   <xacro:wheel name="wheel_4" x="-0.12" y="0.12" z="0.015" rpy="${pi/2}  0 ${pi/4}"/>
-<!--
- <joint name="laser_lidar" type="fixed">
-        <parent link="body" />
-        <child link="lidar" />
-        <origin xyz="0 0 0.103 " rpy="0 -0 0" />
-    </joint>
-    <link name="lidar">
-        <visual>
-            <origin xyz="0.12499999999999995837 -0.12389012757796005748 -0.103" rpy="0 0 0" />
-            <geometry>
-                <mesh filename="package://roboto/robo_description/urdf/chassi/lidar.stl" />
-            </geometry>
-            <material name="lidar_material">
-                <color rgba="1 0 0 1.0" />
-            </material>
-        </visual>
-        <collision>
-            <origin xyz="0.12499999999999995837 -0.12389012757796005748 -0.103" rpy="0 0 0" />
-            <geometry>
-                <mesh filename="package://roboto/robo_description/urdf/chassi/lidar.stl" />
-            </geometry>
-        </collision>
-        <inertial>
-            <mass value="0.1" />
-            <inertia ixx="0.005" ixy="0.0" ixz="0.0" iyy="0.005" iyz="0.0" izz="0.005" />
-        </inertial>
-    </link> -->
 <xacro:include filename="lidar.xacro"/>
+<xacro:include  filename="gazebo.xacro"/>
 </robot>
